File: output/AlcoKeb/AlcoKeb.kicad_pcb (KiCad board)
At the start: 2 copper layers, 150.1 x 113.5 mm, 22 parts

Commit message: Added board constraints and fixed minor things
Routing:
- net P16: track 18.5 -> 150.3 mm
- net P10: track 18.4 -> 132.1 mm
- net P7: track 193.0 -> 186.6 mm
- net GND: track 857.8 -> 864.0 mm
- net P19: track 49.9 -> 45.9 mm
- net P21: track 44.5 -> 48.1 mm
- net P18: track 132.9 -> 129.7 mm
- net P15: track 114.9 -> 112.6 mm
- net P14: track 97.8 -> 95.7 mm
